File: ThunderBuddy.kicad_pcb (KiCad board)
At the start: 2 copper layers, 26.7 x 28.4 mm, 16 parts, among them J1 Headers, U1 AS3935

Commit message: Version 2
Parts:
- added C5: 270pf, Capacitor_SMD:C_0805_2012Metric, F.Cu at (157.8, 92.3)
- C4: renamed from C1; value 1nF -> 680pf
- moved JP3 4.05 mm to (164.6, 98.8)
- moved R3 4.05 mm to (164.6, 101.1)
- moved R4 4.05 mm to (164.6, 99.1)
- moved JP2 4.05 mm to (164.6, 101.4)
- moved C3 3.65 mm to (161.6, 96.1), turned to 90 degrees
- moved R1 2.91 mm to (157.8, 88.3)
- moved C4 1.82 mm to (157.8, 90.3)
- moved JP4 1.15 mm to (154.3, 102.2)
- moved L1 0.21 mm to (157.0, 85.1)
- renumbered C4 to C1
Routing:
- net AD0: track 3.57 -> 9.71 mm
- net GND: track 21.1 -> 15.7 mm
- net AD1: track 3.88 -> 9.21 mm
- net VReg: track 20.0 -> 23.8 mm
- net IN+: track 11.2 -> 13.5 mm
- net SI: track 6.27 -> 8.40 mm
- net Net-(JP4-B): track 3.32 -> 4.51 mm
- net MISO: track 10.1 -> 9.18 mm
- net ACG: track 3.32 -> 4.22 mm
- net MOSI: track 11.2 -> 12.1 mm
- net Vdd: track 18.7 -> 19.5 mm
Other:
- board text added: "V2"
- board text removed: "V1"
