File: ThunderBuddy.kicad_sch (KiCad schematic)
At the start: 16 parts, among them J1 Headers, U1 AS3935

Commit message: Version 2
Parts:
- added C5: 270pf, Capacitor_SMD:C_0805_2012Metric, symbol Device:C_Small
- C4: renamed from C1; value 1nF -> 680pf
- renumbered C4 to C1
Connections:
- net GND: now also C5.2
- net IN+: now also C5.1
Other:
- moved on the sheet: C4, L1, R1
